File: amplifier ckt.sch (EAGLE design)
At the start: 34 parts, among them U1 LM358DR

Commit message: updated ckt
Parts:
- added JP1: (no value), pinhead:PINHD-1X5
- added R17, R18, R19: 1.2k, rcl:R-US_R0603
- added R20: 200k, rcl:R-US_R0603
- added R21: 3k, rcl:R-US_R0603
- added R22: 15k, rcl:R-US_R0603
- added R23: 5.6k, rcl:R-US_R0603
- added X, Y, Z: (no value), pinhead:PINHD-1X1
- C2: device OPL:CAP-POLAR-AVX-B -> rcl:C-USC0805
- R11: value 18k -> 15k
- R12: value 18k -> 3k
- R13: value 220k -> 20k
- R14, R5, R6: value 6.8k -> 5.6k
- R16: value 6.8k -> 1.2k
Connections:
- new net N$20: R17.2, R5.1
- new net N$21: R18.2, R6.1
- new net N$22: R13.2, R20.1
- new net N$23: R16.2, R23.1
- new net N$24: R11.1, R21.2
- new net N$25: R12.2, R22.1
- new net N$26: JP1.3, X.1
- new net N$27: JP1.4, Y.1
- new net N$28: JP1.5, Z.1
- new net N$7: R14.1, R19.2
- net GND: now also C2.1, JP1.2, R17.1, R18.1; no longer C2.+, R5.1, R6.1
- net N$12: now also C2.2; no longer C2.-
- net N$13: now also R21.1, R22.2; no longer R11.1, R12.2
- net N$16: now also R20.2; no longer R13.2
- net N$18: now also R19.1; no longer R14.1
- net VCC: now also JP1.1, R23.2; no longer R16.2
Other:
- moved on the sheet: A2, C5, R11, R12, R13
